Commit message: Add camera to robot model

File: cargobot_description/urdf/cargobot.xacro (robot description, xacro)
@@ -44,4 +44,24 @@
         </inertial>
 	</link>
+    <link name="camera_link">
+		<visual>
+			<origin xyz="0 0 0" rpy="0 0 ${PI/2}" />
+            <geometry>
+                <mesh filename="package://cargobot_description/meshes/camera_link.stl" scale="0.001 0.001 0.001" />
+            </geometry>
+			<material name="Red" />
+		</visual>
+		<collision>
+			<origin xyz="0 0 0" rpy="0 0 ${PI/2}" />
+            <geometry>
+                <mesh filename="package://cargobot_description/meshes/camera_link.stl" scale="0.001 0.001 0.001" />
+            </geometry>
+		</collision>
+        <inertial>
+            <origin xyz="0 0 0" rpy="0 0 0" />
+            <mass value="${mass}" />
+            <inertia ixx="${inertia}" ixy="0.0" ixz="0.0" iyy="${inertia}" iyz="0.0" izz="${inertia}" />
+        </inertial>
+    </link>
     <joint name="base_to_body" type="fixed">
         <axis rpy="0 0 0" xyz="0 0 0"/>
@@ -49,4 +69,10 @@
         <child link="body_link" />
         <origin xyz="0 0 0" rpy="0 0 0"/>
+    </joint>
+    <joint name="camera_to_base" type="fixed">
+        <axis rpy="0 0 0" xyz="0 0 0"/>
+        <parent link="body_link" />
+        <child link="camera_link" />
+        <origin xyz="0.229 0 ${clearance + 0.120}" rpy="0 0 0"/>
     </joint>
     <!-- Wheels -->

Commit message: Add lidar

File: cargobot_description/urdf/cargobot.xacro (robot description, xacro)
@@ -64,4 +64,24 @@
         </inertial>
     </link>
+    <link name="laser">
+        <inertial>
+            <origin xyz="0 0 0" rpy="0 0 0" />
+            <mass value="0.1" />
+            <inertia ixx="0.0" ixy="0.0" ixz="0.0" iyy="0.0" iyz="0.0" izz="0.0" />
+        </inertial>
+        <visual>
+            <origin xyz="0 0 0" rpy="0 0 0" />
+            <geometry>
+                <cylinder radius="0.035" length="0.039"/>
+            </geometry>
+            <material name="Blue" />
+        </visual>
+        <collision>
+            <origin xyz="0 0 0" rpy="0 0 0"/>
+            <geometry>
+                <cylinder radius="0.035" length="0.025"/>
+            </geometry>
+        </collision>
+    </link>
     <joint name="base_to_body" type="fixed">
         <axis rpy="0 0 0" xyz="0 0 0"/>
@@ -75,4 +95,10 @@
         <child link="camera_link" />
         <origin xyz="0.229 0 ${clearance + 0.120}" rpy="0 0 0"/>
+    </joint>
+    <joint name="laser_to_base" type="fixed">
+        <axis rpy="0 0 0" xyz="0 0 0"/>
+        <parent link="body_link" />
+        <child link="laser" />
+        <origin xyz="0 0 ${clearance + 0.16}" rpy="0 0 0"/>
     </joint>
     <!-- Wheels -->
